Commit message: fix rpy parameter order

File: src/inmoov_description/description/example_robot.urdf.xacro (robot description, xacro)
@@ -31,6 +31,6 @@
         <parent link="base" />
         <child link="l3" />
-        <origin  rpy="0 0 0" xyz="0 0.25 0" />
-        <axis rpy="0 0 0" xyz="0 0 1" />
+        <origin xyz="0 0.25 0" rpy="0 0 0"  />
+        <axis xyz="0 0 1" rpy="0 0 0" />
         <limit effort="0.1" lower="-3.1" upper="3.1" velocity="0.2"/>
     </joint>
@@ -48,6 +48,6 @@
         <child link="l2" />
         <!-- <origin xyz="1 0 0" /> -->
-        <origin rpy="0 0 0" xyz="1.5 0 0" />
-        <axis rpy="0 0 0" xyz="0 0 1" />
+        <origin xyz="1.5 0 0" rpy="0 0 0" />
+        <axis xyz="0 0 1" rpy="0 0 0" />
         <limit effort="0.1" lower="-3.1" upper="3.1" velocity="0.2"/>
     </joint>
@@ -64,6 +64,6 @@
         <parent link="l2" />
         <child link="l1" />
-        <origin rpy="0 0 0" xyz="1.5 0 0" />
-        <axis rpy="0 0 0" xyz="0 0 1" />
+        <origin xyz="1.5 0 0" rpy="0 0 0" />
+        <axis xyz="0 0 1" rpy="0 0 0" />
         <limit effort="0.1" lower="-3.1" upper="3.1" velocity="0.2"/>
     </joint>
@@ -80,6 +80,6 @@
         <parent link="l1" />
         <child link="grip" />
-        <origin rpy="0 0 0" xyz="1 0 0" />
-        <axis rpy="0 0 0" xyz="0 0 1" />
+        <origin xyz="1 0 0" rpy="0 0 0" />
+        <axis xyz="0 0 1" rpy="0 0 0" />
         <limit effort="0.1" lower="-3.1" upper="3.1" velocity="0.2"/>
     </joint>
@@ -96,5 +96,5 @@
         <parent link="world" />
         <child link="camera" />
-        <origin  rpy="-2 0 2.5" xyz="4 1 2" />
+        <origin xyz="4 1 2" rpy="-2 0 2.5" />
     </joint>
     <link name="camera">

Commit message: multiple package changes

File: src/inmoov_description/description/example_robot.urdf.xacro (robot description, xacro)
@@ -31,6 +31,6 @@
         <parent link="base" />
         <child link="l3" />
-        <origin xyz="0 0.25 0" rpy="0 0 0"  />
-        <axis xyz="0 0 1" rpy="0 0 0" />
+        <origin  rpy="0 0 0" xyz="0 0.25 0" />
+        <axis rpy="0 0 0" xyz="0 0 1" />
         <limit effort="0.1" lower="-3.1" upper="3.1" velocity="0.2"/>
     </joint>
@@ -48,6 +48,6 @@
         <child link="l2" />
         <!-- <origin xyz="1 0 0" /> -->
-        <origin xyz="1.5 0 0" rpy="0 0 0" />
-        <axis xyz="0 0 1" rpy="0 0 0" />
+        <origin rpy="0 0 0" xyz="1.5 0 0" />
+        <axis rpy="0 0 0" xyz="0 0 1" />
         <limit effort="0.1" lower="-3.1" upper="3.1" velocity="0.2"/>
     </joint>
@@ -64,6 +64,6 @@
         <parent link="l2" />
         <child link="l1" />
-        <origin xyz="1.5 0 0" rpy="0 0 0" />
-        <axis xyz="0 0 1" rpy="0 0 0" />
+        <origin rpy="0 0 0" xyz="1.5 0 0" />
+        <axis rpy="0 0 0" xyz="0 0 1" />
         <limit effort="0.1" lower="-3.1" upper="3.1" velocity="0.2"/>
     </joint>
@@ -80,6 +80,6 @@
         <parent link="l1" />
         <child link="grip" />
-        <origin xyz="1 0 0" rpy="0 0 0" />
-        <axis xyz="0 0 1" rpy="0 0 0" />
+        <origin rpy="0 0 0" xyz="1 0 0" />
+        <axis rpy="0 0 0" xyz="0 0 1" />
         <limit effort="0.1" lower="-3.1" upper="3.1" velocity="0.2"/>
     </joint>
@@ -96,5 +96,5 @@
         <parent link="world" />
         <child link="camera" />
-        <origin xyz="4 1 2" rpy="-2 0 2.5" />
+        <origin  rpy="-2 0 2.5" xyz="4 1 2" />
     </joint>
     <link name="camera">
