Commit message: Many updates and fixes

File: src/inmoov_description/robots/inmoov.urdf.backup.xacro (robot description, xacro)
@@ -14,5 +14,4 @@
 <xacro:include filename="$(find inmoov_description)/urdf/asmArm.urdf.xacro" />
 <xacro:include filename="$(find inmoov_description)/urdf/asmHand.urdf.xacro" />
-<!-- For now we start with a world link.  We might change this later. -->
   <link name="world"/>
   <joint name="fixed" type="fixed">
@@ -58,5 +57,4 @@
      <origin rpy="0 0 0"  xyz="0 0 0"/>
   </joint>
-  <!-- Run macro called "torso" in file asmTorso.urdf.xacro -->
   <xacro:torso covers="yes" />
   <joint name="head_roll_joint" type="revolute">
@@ -74,7 +72,5 @@
    <child link="head_base_link"/>
   </joint>
-  <!-- Run macro called "head" in file asmHead.urdf.xacro -->
   <xacro:head covers="yes" />
-  <!-- Run macro called "face" in file asmFace.urdf.xacro -->
   <xacro:face covers="yes" />
   <joint name="face_joint" type="fixed">
@@ -83,6 +79,4 @@
     <child link="face_link"/>
   </joint>
-  <!-- Run macro called "face" in file asmArm.urdf.xacro -->
-  <!-- We pass the param "side" in order to process 2 arms with 2 hands, right(r) in this case-->
   <xacro:arm side="r" flip="1" covers="yes" />
   <joint name="r_shoulder_out_joint" type="revolute">
@@ -102,6 +96,4 @@
   </joint>
   <xacro:arm side="l" flip="-1" covers="yes" />
-  <!-- Run macro called "face" in file asmArm.urdf.xacro -->
-  <!-- We pass the param "side" in order to process 2 arms with 2 hands, left(l) in this case-->
   <joint name="l_shoulder_out_joint" type="revolute">
    <axis xyz="1 0 0"/>

File: src/inmoov_description/urdf/config.joints.urdf.xacro (robot description, xacro)
@@ -3,5 +3,5 @@
   <xacro:property name="filename" value="$(find inmoov_bringup)/config/config.yaml"/>
   <xacro:property name="c" value="${load_yaml(filename)}"/>
-  xacro:property name="pi" value="3.1415926539"/
+  <xacro:property name="pi" value="3.1415926539"/>
   <xacro:if value="${c['bringup']['angles'] == 'degrees'}">
     <xacro:property name="r" value="${pi/180.0}"/>
