Commit message: update

File: src/inmoov_description/robots/inmoov.urdf (robot description, URDF)
Before this commit: robot robot, 7 links, 6 joints
Links:
- removed link base
- removed link camera
- removed link grip
- removed link l1
- removed link l2
- removed link l3
- added link base_link; visual cylinder length=0.11 radius=0.26
- added link chestplate_link, mass 755.6806875; visual mesh filename=package://inmoov_meshes/meshes/chest.stl scale=0.001 0.001 0.001
- added link disk_link, mass 178.96734375; visual mesh filename=package://inmoov_meshes/meshes/disk.stl scale=0.001 0.001 0.001
- added link eyesupport_link, mass 27.550294922000003; visual mesh filename=package://inmoov_meshes/meshes/eyesupport.stl scale=0.001 0.001 0.001
- added link face_link, mass 46.55903125; visual mesh filename=package://inmoov_meshes/meshes/face.stl scale=0.001 0.001 0.001
- added link head_base_link, mass 43.50228125; visual mesh filename=package://inmoov_meshes/meshes/head_base.stl scale=0.001 0.001 0.001
- added link head_link, mass 120.499460938; visual mesh filename=package://inmoov_meshes/meshes/head.stl scale=0.001 0.001 0.001
- added link head_tilt_link, mass 0.001; visual mesh filename=package://inmoov_meshes/meshes/virtual.stl scale=0.001 0.001 0.001
- added link jaw_link, mass 58.767261719000004; visual mesh filename=package://inmoov_meshes/meshes/jaw.stl scale=0.001 0.001 0.001
- added link kinect2_ir_optical_frame, mass 790.8319375; visual mesh filename=package://inmoov_meshes/meshes/kinectone.stl scale=0.001 0.001 0.001
- added link kinect2_link, mass 790.8319375; visual mesh filename=package://inmoov_meshes/meshes/kinectone.stl scale=0.001 0.001 0.001
- added link kinect2_rgb_optical_frame, mass 790.8319375; visual mesh filename=package://inmoov_meshes/meshes/kinectone.stl scale=0.001 0.001 0.001
- added link l_bicep_link, mass 281.91265625; visual mesh filename=package://inmoov_meshes/meshes/bicep.stl scale=0.001 0.001 0.001
- added link l_bicepcover_link, mass 176.269609375; visual mesh filename=package://inmoov_meshes/meshes/bicepcover.stl scale=0.001 0.001 0.001
- added link l_camera_link, mass 2.4660676269999997; visual mesh filename=package://inmoov_meshes/meshes/camera.stl scale=0.001 0.001 0.001
- added link l_cover_handpinky_link, mass 3.887731445; visual mesh filename=package://inmoov_meshes/meshes/l_cover_handpinky.stl scale=0.001 0.001 0.001
- added link l_cover_handring_link, mass 3.507538086; visual mesh filename=package://inmoov_meshes/meshes/l_cover_handring.stl scale=0.001 0.001 0.001
- added link l_cover_index_link, mass 1.6353686520000001; visual mesh filename=package://inmoov_meshes/meshes/l_cover_index.stl scale=0.001 0.001 0.001
- added link l_cover_middle_link, mass 1.904471313; visual mesh filename=package://inmoov_meshes/meshes/l_cover_middle.stl scale=0.001 0.001 0.001
- added link l_cover_pinky_link, mass 1.2856073; visual mesh filename=package://inmoov_meshes/meshes/l_cover_pinky.stl scale=0.001 0.001 0.001
- added link l_cover_ring_link, mass 1.4669017329999998; visual mesh filename=package://inmoov_meshes/meshes/l_cover_ring.stl scale=0.001 0.001 0.001
- added link l_cover_thumb_link, mass 3.250209717; visual mesh filename=package://inmoov_meshes/meshes/l_cover_thumb.stl scale=0.001 0.001 0.001
- added link l_eye_link, mass 4.659753906; visual mesh filename=package://inmoov_meshes/meshes/eye.stl scale=0.001 0.001 0.001
- added link l_eyesupport_link, mass 11.370105469; visual mesh filename=package://inmoov_meshes/meshes/l_eyesupport.stl scale=0.001 0.001 0.001
- added link l_forearm_link, mass 401.76659375; visual mesh filename=package://inmoov_meshes/meshes/l_forearm.stl scale=0.001 0.001 0.001
- added link l_hand_link, mass 83.605007812; visual mesh filename=package://inmoov_meshes/meshes/l_hand.stl scale=0.001 0.001 0.001
- added link l_handcover_link, mass 39.850039062; visual mesh filename=package://inmoov_meshes/meshes/l_cover_hand.stl scale=0.001 0.001 0.001
- added link l_index1_link, mass 4.8545507809999995; visual mesh filename=package://inmoov_meshes/meshes/index3_1.stl scale=0.001 0.001 0.001
- added link l_index2_link, mass 2.911548828; visual mesh filename=package://inmoov_meshes/meshes/index3_2.stl scale=0.001 0.001 0.001
- added link l_index3_link, mass 2.754759033; visual mesh filename=package://inmoov_meshes/meshes/index3_3.stl scale=0.001 0.001 0.001
- added link l_iris_link, mass 1.026836548; visual mesh filename=package://inmoov_meshes/meshes/iris.stl scale=0.001 0.001 0.001
- added link l_middle1_link, mass 5.988140625; visual mesh filename=package://inmoov_meshes/meshes/middle3_1.stl scale=0.001 0.001 0.001
- added link l_middle2_link, mass 3.588543701; visual mesh filename=package://inmoov_meshes/meshes/middle3_2.stl scale=0.001 0.001 0.001
- added link l_middle3_link, mass 3.395293457; visual mesh filename=package://inmoov_meshes/meshes/middle3_3.stl scale=0.001 0.001 0.001
- added link l_pinky1_link, mass 14.892949219; visual mesh filename=package://inmoov_meshes/meshes/l_pinky3_1.stl scale=0.001 0.001 0.001
- added link l_pinky2_link, mass 3.0539240719999996; visual mesh filename=package://inmoov_meshes/meshes/pinky3_2.stl scale=0.001 0.001 0.001
- added link l_pinky3_link, mass 1.8487075199999998; visual mesh filename=package://inmoov_meshes/meshes/pinky3_3.stl scale=0.001 0.001 0.001
- added link l_pinky4_link, mass 1.7482214360000001; visual mesh filename=package://inmoov_meshes/meshes/pinky3_4.stl scale=0.001 0.001 0.001
- added link l_ring1_link, mass 10.81030957; visual mesh filename=package://inmoov_meshes/meshes/l_ring3_1.stl scale=0.001 0.001 0.001
- added link l_ring2_link, mass 4.222559082; visual mesh filename=package://inmoov_meshes/meshes/ring3_2.stl scale=0.001 0.001 0.001
- added link l_ring3_link, mass 2.530003662; visual mesh filename=package://inmoov_meshes/meshes/ring3_3.stl scale=0.001 0.001 0.001
- added link l_ring4_link, mass 2.3937583009999996; visual mesh filename=package://inmoov_meshes/meshes/ring3_4.stl scale=0.001 0.001 0.001
- added link l_shoulder_base_link, mass 266.52696875; visual mesh filename=package://inmoov_meshes/meshes/l_shoulder_base.stl scale=0.001 0.001 0.001
- added link l_shoulder_link, mass 322.44334375; visual mesh filename=package://inmoov_meshes/meshes/l_shoulder.stl scale=0.001 0.001 0.001
- added link l_thumb1_link, mass 10.0444375; visual mesh filename=package://inmoov_meshes/meshes/l_thumb5_1.stl scale=0.001 0.001 0.001
- added link l_thumb2_link, mass 7.511052246; visual mesh filename=package://inmoov_meshes/meshes/thumb5_2.stl scale=0.001 0.001 0.001
- added link l_thumb3_link, mass 5.812545409999999; visual mesh filename=package://inmoov_meshes/meshes/thumb5_3.stl scale=0.001 0.001 0.001
- added link left_ear_link, mass 85.19796093800001; visual mesh filename=package://inmoov_meshes/meshes/earleftv1.stl scale=0.001 0.001 0.001
- added link mid_stomach_link, mass 1710.217625; visual mesh filename=package://inmoov_meshes/meshes/mid_stomach.stl scale=0.001 0.001 0.001
- added link pedestal_link; visual cylinder length=0.94 radius=0.0254
- added link r_bicep_link, mass 281.91265625; visual mesh filename=package://inmoov_meshes/meshes/bicep.stl scale=0.001 0.001 0.001
- added link r_bicepcover_link, mass 176.269609375; visual mesh filename=package://inmoov_meshes/meshes/bicepcover.stl scale=0.001 0.001 0.001
- added link r_camera_link, mass 2.4660676269999997; visual mesh filename=package://inmoov_meshes/meshes/camera.stl scale=0.001 0.001 0.001
- added link r_cover_handpinky_link, mass 3.887731445; visual mesh filename=package://inmoov_meshes/meshes/r_cover_handpinky.stl scale=0.001 0.001 0.001
- added link r_cover_handring_link, mass 3.50753833; visual mesh filename=package://inmoov_meshes/meshes/r_cover_handring.stl scale=0.001 0.001 0.001
- added link r_cover_index_link, mass 1.6353686520000001; visual mesh filename=package://inmoov_meshes/meshes/r_cover_index.stl scale=0.001 0.001 0.001
- added link r_cover_middle_link, mass 1.904471313; visual mesh filename=package://inmoov_meshes/meshes/r_cover_middle.stl scale=0.001 0.001 0.001
- added link r_cover_pinky_link, mass 1.2856073; visual mesh filename=package://inmoov_meshes/meshes/r_cover_pinky.stl scale=0.001 0.001 0.001
- added link r_cover_ring_link, mass 1.4669017329999998; visual mesh filename=package://inmoov_meshes/meshes/r_cover_ring.stl scale=0.001 0.001 0.001
- added link r_cover_thumb_link, mass 3.250209961; visual mesh filename=package://inmoov_meshes/meshes/r_cover_thumb.stl scale=0.001 0.001 0.001
- added link r_eye_link, mass 4.659753906; visual mesh filename=package://inmoov_meshes/meshes/eye.stl scale=0.001 0.001 0.001
- added link r_eyesupport_link, mass 11.370105469; visual mesh filename=package://inmoov_meshes/meshes/r_eyesupport.stl scale=0.001 0.001 0.001
- added link r_forearm_link, mass 401.76659375; visual mesh filename=package://inmoov_meshes/meshes/r_forearm.stl scale=0.001 0.001 0.001
- added link r_hand_link, mass 83.605; visual mesh filename=package://inmoov_meshes/meshes/r_hand.stl scale=0.001 0.001 0.001
- added link r_handcover_link, mass 39.850042969; visual mesh filename=package://inmoov_meshes/meshes/r_cover_hand.stl scale=0.001 0.001 0.001
- added link r_index1_link, mass 4.8545507809999995; visual mesh filename=package://inmoov_meshes/meshes/index3_1.stl scale=0.001 0.001 0.001
- added link r_index2_link, mass 2.911548828; visual mesh filename=package://inmoov_meshes/meshes/index3_2.stl scale=0.001 0.001 0.001
- added link r_index3_link, mass 2.754759033; visual mesh filename=package://inmoov_meshes/meshes/index3_3.stl scale=0.001 0.001 0.001
- added link r_iris_link, mass 1.026836548; visual mesh filename=package://inmoov_meshes/meshes/iris.stl scale=0.001 0.001 0.001
- added link r_middle1_link, mass 5.988140625; visual mesh filename=package://inmoov_meshes/meshes/middle3_1.stl scale=0.001 0.001 0.001
- added link r_middle2_link, mass 3.588543701; visual mesh filename=package://inmoov_meshes/meshes/middle3_2.stl scale=0.001 0.001 0.001
- added link r_middle3_link, mass 3.395293457; visual mesh filename=package://inmoov_meshes/meshes/middle3_3.stl scale=0.001 0.001 0.001
- added link r_pinky1_link, mass 14.892949219; visual mesh filename=package://inmoov_meshes/meshes/r_pinky3_1.stl scale=0.001 0.001 0.001
- added link r_pinky2_link, mass 3.0539240719999996; visual mesh filename=package://inmoov_meshes/meshes/pinky3_2.stl scale=0.001 0.001 0.001
- added link r_pinky3_link, mass 1.8487075199999998; visual mesh filename=package://inmoov_meshes/meshes/pinky3_3.stl scale=0.001 0.001 0.001
- added link r_pinky4_link, mass 1.7482214360000001; visual mesh filename=package://inmoov_meshes/meshes/pinky3_4.stl scale=0.001 0.001 0.001
- added link r_ring1_link, mass 10.81030957; visual mesh filename=package://inmoov_meshes/meshes/r_ring3_1.stl scale=0.001 0.001 0.001
- added link r_ring2_link, mass 4.222559082; visual mesh filename=package://inmoov_meshes/meshes/ring3_2.stl scale=0.001 0.001 0.001
- added link r_ring3_link, mass 2.530003662; visual mesh filename=package://inmoov_meshes/meshes/ring3_3.stl scale=0.001 0.001 0.001
- added link r_ring4_link, mass 2.3937583009999996; visual mesh filename=package://inmoov_meshes/meshes/ring3_4.stl scale=0.001 0.001 0.001
- added link r_shoulder_base_link, mass 266.52696875; visual mesh filename=package://inmoov_meshes/meshes/r_shoulder_base.stl scale=0.001 0.001 0.001
- added link r_shoulder_link, mass 322.44334375; visual mesh filename=package://inmoov_meshes/meshes/r_shoulder.stl scale=0.001 0.001 0.001
- added link r_thumb1_link, mass 10.044436523; visual mesh filename=package://inmoov_meshes/meshes/r_thumb5_1.stl scale=0.001 0.001 0.001
- added link r_thumb2_link, mass 7.511052246; visual mesh filename=package://inmoov_meshes/meshes/thumb5_2.stl scale=0.001 0.001 0.001
- added link r_thumb3_link, mass 5.812545409999999; visual mesh filename=package://inmoov_meshes/meshes/thumb5_3.stl scale=0.001 0.001 0.001
- added link right_ear_link, mass 85.17540625; visual mesh filename=package://inmoov_meshes/meshes/earrightv1.stl scale=0.001 0.001 0.001
- added link skull_link, mass 422.3130625; visual mesh filename=package://inmoov_meshes/meshes/skull.stl scale=0.001 0.001 0.001
- added link top_stomach_link, mass 1144.88975; visual mesh filename=package://inmoov_meshes/meshes/top_stomach.stl scale=0.001 0.001 0.001
- added link torso_link, mass 1923.29375; visual mesh filename=package://inmoov_meshes/meshes/torso.stl scale=0.001 0.001 0.001
Joints:
- removed joint base_to_l3
- removed joint l1_to_grip
- removed joint l2_to_l1
- removed joint l3_to_l2
- removed joint world_to_base
- removed joint world_to_camera
- added joint base_to_pedestal_link: type fixed, parent base_link, child pedestal_link, origin xyz=0 0 0 rpy=0 0 0
- added joint chestplate_joint: type fixed, parent torso_link, child chestplate_link, origin xyz=0.042 0 0.025 rpy=0 0 0
- added joint disk_joint: type fixed, parent top_stomach_link, child disk_link, origin xyz=0.046 0 0.09 rpy=0 0 0
- added joint eyes_pan_joint: type revolute, parent eyesupport_link, child r_eyesupport_link, origin xyz=0 0.033 -0.0036 rpy=0 0 0, axis 0 0 1, limit lower=-0.5235987755982988 upper=0.5235987755982988 effort=1000.0 velocity=0.0
- added joint eyes_tilt_joint: type revolute, parent face_link, child eyesupport_link, origin xyz=0 0 0 rpy=0 0 0, axis 0 1 0, limit lower=0.2617993877991494 upper=-0.2617993877991494 effort=1000.0 velocity=0.0
- added joint face_joint: type fixed, parent skull_link, child face_link, origin xyz=0.0637 0 0.079 rpy=0 0 0
- added joint fixed: type fixed, parent world, child base_link
- added joint head_pan_joint: type revolute, parent head_base_link, child head_link, origin xyz=0 0 0.0245 rpy=0 0 0, axis 0 0 1, limit lower=-1.7453292519943295 upper=1.5707963267948966 effort=1000.0 velocity=0.0
- added joint head_roll_joint: type revolute, parent torso_link, child head_tilt_link, origin xyz=-0.0315  -0.001 0.4551 rpy=0 0 3.1415, axis 1 0 0, limit lower=-0.2617993877991494 upper=0.2617993877991494 effort=1000.0 velocity=0.0
- added joint head_tilt_joint: type revolute, parent head_tilt_link, child head_base_link, origin xyz=0 0 0 rpy=0 0 3.1415, axis 0 1 0, limit lower=-0.3490658503988659 upper=0.3490658503988659 effort=1000.0 velocity=0.0
- added joint jaw_joint: type revolute, parent head_link, child jaw_link, origin xyz=0.0375 0.0005 0.0437 rpy=0 0.09 0, axis 0 1 0, limit lower=0.0 upper=0.08726646259971647 effort=1000.0 velocity=0.0
- added joint kinect2_ir_optical_frame_joint: type fixed, parent torso_link, child kinect2_ir_optical_frame, origin xyz=0 0 0.066 rpy=-1.57 0 -1.57
- added joint kinect2_joint: type fixed, parent torso_link, child kinect2_link, origin xyz=0 0 0.066 rpy=-1.57 0 -1.57
- added joint kinect2_rgb_optical_joint: type fixed, parent torso_link, child kinect2_rgb_optical_frame, origin xyz=0 0 0.066 rpy=-1.57 0 -1.57
- added joint l_bicepcover_joint: type fixed, parent l_bicep_link, child l_bicepcover_link, origin xyz=0 0 0 rpy=0 0 0
- added joint l_camera_joint: type fixed, parent l_eyesupport_link, child l_camera_link, origin xyz=-0.001 0 0 rpy=0 0 0
- added joint l_cover_handpinky_joint: type fixed, parent l_pinky1_link, child l_cover_handpinky_link, origin xyz=0.01 0.02025 -0.0071 rpy=0.7 0 0
- added joint l_cover_handring_joint: type fixed, parent l_ring1_link, child l_cover_handring_link, origin xyz=0.009 0.015 -0.0008 rpy=0.7 0 0
- added joint l_cover_index_joint: type fixed, parent l_index1_link, child l_cover_index_link, origin xyz=0.0071 0 -0.012 rpy=0 -0.05 0
- added joint l_cover_middle_joint: type fixed, parent l_middle1_link, child l_cover_middle_link, origin xyz=0.0071 0 -0.012 rpy=0 0.05 0
- added joint l_cover_pinky_joint: type fixed, parent l_pinky2_link, child l_cover_pinky_link, origin xyz=0.005 0 -0.0105 rpy=-0.1 0.05 0
- added joint l_cover_ring_joint: type fixed, parent l_ring2_link, child l_cover_ring_link, origin xyz=0.005 0 -0.011 rpy=-0.1 0.05 0
- added joint l_cover_thumb_joint: type fixed, parent l_thumb1_link, child l_cover_thumb_link, origin xyz=0.01 -0.02125 0.0047 rpy=-0.05 0 0
- added joint l_elbow_flex_joint: type revolute, parent l_bicep_link, child l_forearm_link, origin xyz=-0.0278 0 -0.2235 rpy=0 0 0, axis 0 1 0, limit lower=-0.2617993877991494 upper=-1.4835298641951802 effort=1000.0 velocity=0.0
- added joint l_eye_joint: type fixed, parent l_eyesupport_link, child l_eye_link, origin xyz=0.003 0 0 rpy=0 0 0
- added joint l_eye_pan_joint: type revolute, parent eyesupport_link, child l_eyesupport_link, origin xyz=0 -0.033 -0.0036 rpy=0 0 0, axis 0 0 1, limit lower=-0.5235987755982988 upper=0.5235987755982988 effort=1000.0 velocity=0.0, mimic joint=eyes_pan_joint multiplier=1 offset=0
- added joint l_handcover_joint: type fixed, parent l_hand_link, child l_handcover_link, origin xyz=0.009 -0.0192 -0.0977 rpy=0 0 0
- added joint l_index1_joint: type revolute, parent l_hand_link, child l_index1_link, origin xyz=-0.0015 -0.0342  -0.119 rpy=-0.1 0 0, axis 0 1 0, limit lower=-0.08726646259971647 upper=1.4835298641951802 effort=1000.0 velocity=0.0, mimic joint=l_index_joint multiplier=1 offset=0
- added joint l_index3_joint: type revolute, parent l_index2_link, child l_index3_link, origin xyz=0 0 -0.024 rpy=0 0 0, axis 0 1 0, limit lower=-0.08726646259971647 upper=1.4835298641951802 effort=1000.0 velocity=0.0, mimic joint=l_index_joint multiplier=1 offset=0
- added joint l_index_joint: type revolute, parent l_index1_link, child l_index2_link, origin xyz=0 0.001 -0.03595 rpy=0 0 0, axis 0 1 0, limit lower=-0.08726646259971647 upper=1.4835298641951802 effort=1000.0 velocity=0.0
- added joint l_iris_joint: type fixed, parent l_eyesupport_link, child l_iris_link, origin xyz=0.0061 0 0 rpy=0 0 0
- added joint l_middle1_joint: type revolute, parent l_hand_link, child l_middle1_link, origin xyz=-0.00175 -0.007  -0.12325 rpy=0 0 0, axis 0 1 0, limit lower=-0.08726646259971647 upper=1.4835298641951802 effort=1000.0 velocity=0.0, mimic joint=l_middle_joint multiplier=1 offset=0
- added joint l_middle3_joint: type revolute, parent l_middle2_link, child l_middle3_link, origin xyz=0 0.0005 -0.0259 rpy=0 0 0, axis 0 1 0, limit lower=-0.08726646259971647 upper=1.4835298641951802 effort=1000.0 velocity=0.0, mimic joint=l_middle_joint multiplier=1 offset=0
- added joint l_middle_joint: type revolute, parent l_middle1_link, child l_middle2_link, origin xyz=0 0.000 -0.0389 rpy=0 0 0, axis 0 1 0, limit lower=-0.08726646259971647 upper=1.4835298641951802 effort=1000.0 velocity=0.0
- added joint l_pinky1_joint: type revolute, parent l_hand_link, child l_pinky1_link, origin xyz=0 0.027 -0.0555 rpy=-0.7 0 0, axis 0 0 1, limit lower=-0.08726646259971647 upper=1.4835298641951802 effort=1000.0 velocity=0.0, mimic joint=l_pinky_joint multiplier=0.1 offset=0
- added joint l_pinky3_joint: type revolute, parent l_pinky2_link, child l_pinky3_link, origin xyz=0 0.0005 -0.031 rpy=0 0 0, axis 0 1 0, limit lower=-0.08726646259971647 upper=1.4835298641951802 effort=1000.0 velocity=0.0, mimic joint=l_pinky_joint multiplier=1 offset=0
- added joint l_pinky4_joint: type revolute, parent l_pinky3_link, child l_pinky4_link, origin xyz=0 0.0004 -0.0208 rpy=0 0 0, axis 0 1 0, limit lower=-0.08726646259971647 upper=1.4835298641951802 effort=1000.0 velocity=0.0, mimic joint=l_pinky_joint multiplier=1 offset=0
- added joint l_pinky_joint: type revolute, parent l_pinky1_link, child l_pinky2_link, origin xyz=0 0.046 -0.0228 rpy=0.93 0 0, axis 0 1 0, limit lower=-0.08726646259971647 upper=1.4835298641951802 effort=1000.0 velocity=0.0
- added joint l_ring1_joint: type revolute, parent l_hand_link, child l_ring1_link, origin xyz=0 0.00705 -0.0794 rpy=-0.7 0 0, axis 0 0 1, limit lower=-0.08726646259971647 upper=1.4835298641951802 effort=1000.0 velocity=0.0, mimic joint=l_ring_joint multiplier=0.1 offset=0
- added joint l_ring3_joint: type revolute, parent l_ring2_link, child l_ring3_link, origin xyz=0 0.0005 -0.0345 rpy=0 0 0, axis 0 1 0, limit lower=-0.08726646259971647 upper=1.4835298641951802 effort=1000.0 velocity=0.0, mimic joint=l_ring_joint multiplier=1 offset=0
- added joint l_ring4_joint: type revolute, parent l_ring3_link, child l_ring4_link, origin xyz=0 0.0004 -0.0229 rpy=0 0 0, axis 0 1 0, limit lower=-0.08726646259971647 upper=1.4835298641951802 effort=1000.0 velocity=0.0, mimic joint=l_ring_joint multiplier=1 offset=0
- added joint l_ring_joint: type revolute, parent l_ring1_link, child l_ring2_link, origin xyz=0.00126 0.0351 -0.0166 rpy=0.7775 0 0, axis 0 1 0, limit lower=-0.08726646259971647 upper=1.4835298641951802 effort=1000.0 velocity=0.0
- added joint l_shoulder_lift_joint: type revolute, parent l_shoulder_base_link, child l_shoulder_link, origin xyz=0 0.012 -0.04 rpy=0 0 0, axis 0 1 0, limit lower=0.7853981633974483 upper=-2.356194490192345 effort=1000.0 velocity=0.0
- added joint l_shoulder_out_joint: type revolute, parent torso_link, child l_shoulder_base_link, origin xyz=0 0.143 0.298 rpy=0 0 0, axis 1 0 0, limit lower=0.08726646259971647 upper=1.0471975511965976 effort=1000.0 velocity=0.0
- added joint l_thumb1_joint: type revolute, parent l_hand_link, child l_thumb1_link, origin xyz=0 -0.029 -0.0577 rpy=-0.1 0 0, axis 0 0 1, limit lower=-0.08726646259971647 upper=1.1344640137963142 effort=1000.0 velocity=0.0, mimic joint=l_thumb_joint multiplier=-0.75 offset=0
- added joint l_thumb3_joint: type revolute, parent l_thumb2_link, child l_thumb3_link, origin xyz=0 0 -0.035 rpy=0 0 0, axis 0 1 0, limit lower=-0.08726646259971647 upper=1.1344640137963142 effort=1000.0 velocity=0.0, mimic joint=l_thumb_joint multiplier=1 offset=0
- added joint l_thumb_joint: type revolute, parent l_thumb1_link, child l_thumb2_link, origin xyz=-0.00052 -0.02725  -0.013 rpy=-0.825 -0.1 -0.3, axis 0 1 0, limit lower=-0.08726646259971647 upper=1.1344640137963142 effort=1000.0 velocity=0.0
- added joint l_upper_arm_roll_joint: type revolute, parent l_shoulder_link, child l_bicep_link, origin xyz=0 0.066 -0.060 rpy=0 0 0, axis 0 0 1, limit lower=-1.5707963267948966 upper=1.5707963267948966 effort=1000.0 velocity=0.0
- added joint l_wrist_roll_joint: type revolute, parent l_forearm_link, child l_hand_link, origin xyz=-0.0144 -0.01  -0.2885 rpy=0 0 0, axis 0 0 1, limit lower=3.141592653589793 upper=0.0 effort=1000.0 velocity=0.0
- added joint left_ear_joint: type fixed, parent head_link, child left_ear_link, origin xyz=0.035 0.056 0.0437 rpy=0 0 0
- added joint pedestal_to_mid_stomach_joint: type fixed, parent pedestal_link, child mid_stomach_link, origin xyz=0 0 0 rpy=0 0 0
- added joint r_bicepcover_joint: type fixed, parent r_bicep_link, child r_bicepcover_link, origin xyz=0 0 0 rpy=0 0 0
- added joint r_camera_joint: type fixed, parent r_eyesupport_link, child r_camera_link, origin xyz=-0.001 0 0 rpy=0 0 0
- added joint r_cover_handpinky_joint: type fixed, parent r_pinky1_link, child r_cover_handpinky_link, origin xyz=0.01 -0.02025 -0.0071 rpy=-0.7 0 0
- added joint r_cover_handring_joint: type fixed, parent r_ring1_link, child r_cover_handring_link, origin xyz=0.009 -0.015 -0.0008 rpy=-0.7 0 0
- added joint r_cover_index_joint: type fixed, parent r_index1_link, child r_cover_index_link, origin xyz=0.0071 0 -0.012 rpy=0 0.05 0
- added joint r_cover_middle_joint: type fixed, parent r_middle1_link, child r_cover_middle_link, origin xyz=0.0071 0 -0.012 rpy=0 -0.05 0
- added joint r_cover_pinky_joint: type fixed, parent r_pinky2_link, child r_cover_pinky_link, origin xyz=0.005 0 -0.0105 rpy=0.1 -0.05 0
- added joint r_cover_ring_joint: type fixed, parent r_ring2_link, child r_cover_ring_link, origin xyz=0.005 0 -0.011 rpy=0.1 -0.05 0
- added joint r_cover_thumb_joint: type fixed, parent r_thumb1_link, child r_cover_thumb_link, origin xyz=0.01 0.02125 0.0047 rpy=0.05 0 0
- added joint r_elbow_flex_joint: type revolute, parent r_bicep_link, child r_forearm_link, origin xyz=-0.0278 0 -0.2235 rpy=0 0 0, axis 0 1 0, limit lower=-0.2617993877991494 upper=-1.3962634015954636 effort=1000.0 velocity=0.0
- added joint r_eye_joint: type fixed, parent r_eyesupport_link, child r_eye_link, origin xyz=0.003 0 0 rpy=0 0 0
- added joint r_handcover_joint: type fixed, parent r_hand_link, child r_handcover_link, origin xyz=0.009 0.0192 -0.0977 rpy=0 0 0
- added joint r_index1_joint: type revolute, parent r_hand_link, child r_index1_link, origin xyz=-0.0015 0.0342  -0.119 rpy=0.1 0 0, axis 0 1 0, limit lower=-0.08726646259971647 upper=1.4835298641951802 effort=1000.0 velocity=0.0, mimic joint=r_index_joint multiplier=1 offset=0
- added joint r_index3_joint: type revolute, parent r_index2_link, child r_index3_link, origin xyz=0 0 -0.024 rpy=0 0 0, axis 0 1 0, limit lower=-0.08726646259971647 upper=1.4835298641951802 effort=1000.0 velocity=0.0, mimic joint=r_index_joint multiplier=1 offset=0
- added joint r_index_joint: type revolute, parent r_index1_link, child r_index2_link, origin xyz=0 0.001 -0.03595 rpy=0 0 0, axis 0 1 0, limit lower=-0.08726646259971647 upper=1.4835298641951802 effort=1000.0 velocity=0.0
- added joint r_iris_joint: type fixed, parent r_eyesupport_link, child r_iris_link, origin xyz=0.0061 0 0 rpy=0 0 0
- added joint r_middle1_joint: type revolute, parent r_hand_link, child r_middle1_link, origin xyz=-0.00175 0.007  -0.12325 rpy=0 0 0, axis 0 1 0, limit lower=-0.08726646259971647 upper=1.4835298641951802 effort=1000.0 velocity=0.0, mimic joint=r_middle_joint multiplier=1 offset=0
- added joint r_middle3_joint: type revolute, parent r_middle2_link, child r_middle3_link, origin xyz=0 0.0005 -0.0259 rpy=0 0 0, axis 0 1 0, limit lower=-0.08726646259971647 upper=1.4835298641951802 effort=1000.0 velocity=0.0, mimic joint=r_middle_joint multiplier=1 offset=0
- added joint r_middle_joint: type revolute, parent r_middle1_link, child r_middle2_link, origin xyz=0 0.000 -0.0389 rpy=0 0 0, axis 0 1 0, limit lower=-0.08726646259971647 upper=1.4835298641951802 effort=1000.0 velocity=0.0
- added joint r_pinky1_joint: type revolute, parent r_hand_link, child r_pinky1_link, origin xyz=0 -0.027 -0.0555 rpy=0.7 0 0, axis 0 0 1, limit lower=-0.08726646259971647 upper=1.4835298641951802 effort=1000.0 velocity=0.0, mimic joint=r_pinky_joint multiplier=-0.1 offset=0
- added joint r_pinky3_joint: type revolute, parent r_pinky2_link, child r_pinky3_link, origin xyz=0 0.0005 -0.031 rpy=0 0 0, axis 0 1 0, limit lower=-0.08726646259971647 upper=1.4835298641951802 effort=1000.0 velocity=0.0, mimic joint=r_pinky_joint multiplier=1 offset=0
- added joint r_pinky4_joint: type revolute, parent r_pinky3_link, child r_pinky4_link, origin xyz=0 0.0004 -0.0208 rpy=0 0 0, axis 0 1 0, limit lower=-0.08726646259971647 upper=1.4835298641951802 effort=1000.0 velocity=0.0, mimic joint=r_pinky_joint multiplier=1 offset=0
- added joint r_pinky_joint: type revolute, parent r_pinky1_link, child r_pinky2_link, origin xyz=0 -0.046 -0.0228 rpy=-0.93 0 0, axis 0 1 0, limit lower=-0.08726646259971647 upper=1.4835298641951802 effort=1000.0 velocity=0.0
- added joint r_ring1_joint: type revolute, parent r_hand_link, child r_ring1_link, origin xyz=0 -0.00705 -0.0794 rpy=0.7 0 0, axis 0 0 1, limit lower=-0.08726646259971647 upper=1.4835298641951802 effort=1000.0 velocity=0.0, mimic joint=r_ring_joint multiplier=-0.1 offset=0
- added joint r_ring3_joint: type revolute, parent r_ring2_link, child r_ring3_link, origin xyz=0 0.0005 -0.0345 rpy=0 0 0, axis 0 1 0, limit lower=-0.08726646259971647 upper=1.4835298641951802 effort=1000.0 velocity=0.0, mimic joint=r_ring_joint multiplier=1 offset=0
- added joint r_ring4_joint: type revolute, parent r_ring3_link, child r_ring4_link, origin xyz=0 0.0004 -0.0229 rpy=0 0 0, axis 0 1 0, limit lower=-0.08726646259971647 upper=1.4835298641951802 effort=1000.0 velocity=0.0, mimic joint=r_ring_joint multiplier=1 offset=0
- added joint r_ring_joint: type revolute, parent r_ring1_link, child r_ring2_link, origin xyz=0.00126 -0.0351 -0.0166 rpy=-0.7775 0 0, axis 0 1 0, limit lower=-0.08726646259971647 upper=1.4835298641951802 effort=1000.0 velocity=0.0
- added joint r_shoulder_lift_joint: type revolute, parent r_shoulder_base_link, child r_shoulder_link, origin xyz=0 -0.012 -0.04 rpy=0 0 0, axis 0 1 0, limit lower=0.7853981633974483 upper=-2.356194490192345 effort=1000.0 velocity=0.0
- added joint r_shoulder_out_joint: type revolute, parent torso_link, child r_shoulder_base_link, origin xyz=0 -0.143 0.298 rpy=0 0 0, axis 1 0 0, limit lower=-0.08726646259971647 upper=-1.0471975511965976 effort=1000.0 velocity=0.0
- added joint r_thumb1_joint: type revolute, parent r_hand_link, child r_thumb1_link, origin xyz=0 0.029 -0.0577 rpy=0.1 0 0, axis 0 0 1, limit lower=-0.08726646259971647 upper=1.1344640137963142 effort=1000.0 velocity=0.0, mimic joint=r_thumb_joint multiplier=0.75 offset=0
- added joint r_thumb3_joint: type revolute, parent r_thumb2_link, child r_thumb3_link, origin xyz=0 0 -0.035 rpy=0 0 0, axis 0 1 0, limit lower=-0.08726646259971647 upper=1.1344640137963142 effort=1000.0 velocity=0.0, mimic joint=r_thumb_joint multiplier=1 offset=0
- added joint r_thumb_joint: type revolute, parent r_thumb1_link, child r_thumb2_link, origin xyz=-0.00052 0.02725  -0.013 rpy=0.825 -0.1 0.3, axis 0 1 0, limit lower=-0.08726646259971647 upper=1.1344640137963142 effort=1000.0 velocity=0.0
- added joint r_upper_arm_roll_joint: type revolute, parent r_shoulder_link, child r_bicep_link, origin xyz=0 -0.066 -0.060 rpy=0 0 0, axis 0 0 1, limit lower=1.5707963267948966 upper=-1.5707963267948966 effort=1000.0 velocity=0.0
- added joint r_wrist_roll_joint: type revolute, parent r_forearm_link, child r_hand_link, origin xyz=-0.0144 0.01  -0.2885 rpy=0 0 0, axis 0 0 1, limit lower=0.0 upper=-3.141592653589793 effort=1000.0 velocity=0.0
- added joint right_ear_joint: type fixed, parent head_link, child right_ear_link, origin xyz=0.035 -0.056 0.0437 rpy=0 0 0
- added joint skull_joint: type fixed, parent head_link, child skull_link, origin xyz=0.044 0 -0.0245 rpy=0 0 0
- added joint waist_pan_joint: type revolute, parent mid_stomach_link, child top_stomach_link, origin xyz=0 0 1.152 rpy=0 0 0, axis 0 0 1, limit lower=-1.5707963267948966 upper=1.5707963267948966 effort=1000.0 velocity=0.0
- added joint waist_roll_joint: type revolute, parent top_stomach_link, child torso_link, origin xyz=0 0 0.11 rpy=0 0 0, axis 1 0 0, limit lower=0.2617993877991494 upper=-0.2617993877991494 effort=1000.0 velocity=0.0
