Commit message: launcher and urdf chang es

File: src/inmoov_description/robots/example_robot.urdf.xacro (robot description, xacro)
@@ -17,5 +17,5 @@
         <parent link="world" />
         <child link="base" />
-        <origin  rpy="1.57 0 0" xyz="0 0 0" />
+        <origin xyz="0 0 0" rpy="1.57 0 0" />
     </joint>
     <link name="base">

Commit message: multiple updates

File: src/inmoov_description/robots/example_robot.urdf.xacro (robot description, xacro)
@@ -20,4 +20,8 @@
     </joint>
     <link name="base">
+        <inertial>
+            <mass value="0.001" />
+            <inertia ixx="0.001" ixy="0"  ixz="0" iyy="0.001" iyz="0" izz="0.001" />
+        </inertial>
         <visual>
             <origin xyz="2 0 0" rpy="0 0 0"/>
@@ -32,8 +36,12 @@
         <child link="l3" />
         <origin  rpy="0 0 0" xyz="0 0.25 0" />
-        <axis rpy="0 0 0" xyz="0 0 1" />
+        <!-- <axis rpy="0 0 0" xyz="0 0 1" /> -->
         <limit effort="0.1" lower="-3.1" upper="3.1" velocity="0.2"/>
     </joint>
     <link name="l3">
+        <inertial>
+            <mass value="0.001" />
+            <inertia ixx="0.001" ixy="0"  ixz="0" iyy="0.001" iyz="0" izz="0.001" />
+        </inertial>
         <visual>
             <origin xyz="0.75 0 0" rpy="0 1.57 0"/>

File: src/inmoov_description/robots/inmoov.broke.urdf.xacro (robot description, xacro)
@@ -14,4 +14,11 @@
 <xacro:include filename="$(find inmoov_description)/urdf/asmArm.urdf.xacro" />
 <xacro:include filename="$(find inmoov_description)/urdf/asmHand.urdf.xacro" />
+<!-- For now we start with a world link.  This is because we have no legs yet -->
+<!-- We are basically treating this as a stationary robot with a solid base -->
+<!-- rather than a mobile robot.  A mobile robot will start with a "base_link" instead -->
+<!-- The source I copied already has a base_link.  Maybe we start there later. -->
+<!-- For now we will leave it as part of the robot and leave world as well  -->
+<!-- We will change this later. -->
+<!--  -->
   <link name="world"/>
   <joint name="fixed" type="fixed">
@@ -20,4 +27,14 @@
   </joint>
   <link name="base_link">
+    <inertial>
+      <mass value="58.767261719000004"/>
+      <inertia ixx="0.147272256" ixy="7.553278125e-05" ixz="0.055060208" iyy="0.134112088" iyz="-1.2159836913999999e-05" izz="0.156998304"/>
+    </inertial>
+    <collision>
+      <origin rpy="0 0 0" xyz="0 0 0.055"/>
+      <geometry>
+        <cylinder length="0.11" radius="0.26"/>
+      </geometry>
+    </collision>
     <visual>
       <geometry>
@@ -34,11 +51,21 @@
   </joint>
   <link name="pedestal_link">
+    <collision>
+      <origin xyz="0 0 0" rpy"0 0 0"/>
+      <geometry>
+        <cylinder length="0.11" radius="0.26"/>
+      </geometry>
+    </collision>
     <visual>
       <geometry>
-        <cylinder length="0.94" radius="0.0254"/>
+        <cylinder length="0.11" radius="0.26"/>
       </geometry>
-      <origin rpy="0 0 0" xyz="0 0 0.58"/>
+      <origin rpy="0 0 0" xyz="0 0 0.055"/>
       <xacro:base_color/>
     </visual>
+    <inertial>
+      <mass value="58.767261719000004"/>
+      <inertia ixx="0.147272256" ixy="7.553278125e-05" ixz="0.055060208" iyy="0.134112088" iyz="-1.2159836913999999e-05" izz="0.156998304"/>
+    </inertial>
   </link>
   <link name="head_tilt_link">
@@ -57,4 +84,5 @@
      <origin rpy="0 0 0"  xyz="0 0 0"/>
   </joint>
+  <!-- Run macro called "torso" in file asmTorso.urdf.xacro -->
   <xacro:torso covers="yes" />
   <joint name="head_roll_joint" type="revolute">
@@ -72,5 +100,7 @@
    <child link="head_base_link"/>
   </joint>
+  <!-- Run macro called "head" in file asmHead.urdf.xacro -->
   <xacro:head covers="yes" />
+  <!-- Run macro called "face" in file asmFace.urdf.xacro -->
   <xacro:face covers="yes" />
   <joint name="face_joint" type="fixed">
@@ -79,4 +109,6 @@
     <child link="face_link"/>
   </joint>
+  <!-- Run macro called "face" in file asmArm.urdf.xacro -->
+  <!-- We pass the param "side" in order to process 2 arms with 2 hands, right(r) in this case-->
   <xacro:arm side="r" flip="1" covers="yes" />
   <joint name="r_shoulder_out_joint" type="revolute">
@@ -96,4 +128,6 @@
   </joint>
   <xacro:arm side="l" flip="-1" covers="yes" />
+  <!-- Run macro called "face" in file asmArm.urdf.xacro -->
+  <!-- We pass the param "side" in order to process 2 arms with 2 hands, left(l) in this case-->
   <joint name="l_shoulder_out_joint" type="revolute">
    <axis xyz="1 0 0"/>

File: src/inmoov_description/robots/inmoov.urdf.backup2.xacro (robot description, xacro)
@@ -6,11 +6,19 @@
 <xacro:include filename="$(find inmoov_description)/urdf/inmoov.gazebo" />
 <!-- The following includes are for the various appendages -->
-<!-- <xacro:include filename="$(find inmoov_description)/urdf/asmBase.urdf.xacro" /> -->
+<xacro:include filename="$(find inmoov_description)/urdf/materials.urdf.xacro" />
+<xacro:include filename="$(find inmoov_description)/urdf/asmBase.urdf.xacro" />
 <xacro:include filename="$(find inmoov_description)/urdf/asmTorso.urdf.xacro" />
-<!-- <xacro:include filename="$(find inmoov_description)/urdf/asmHead.urdf.xacro" /> -->
-<!-- <xacro:include filename="$(find inmoov_description)/urdf/asmEye.urdf.xacro" /> -->
-<!-- <xacro:include filename="$(find inmoov_description)/urdf/asmFace.urdf.xacro" /> -->
-<!-- <xacro:include filename="$(find inmoov_description)/urdf/asmArm.urdf.xacro" /> -->
-<!-- <xacro:include filename="$(find inmoov_description)/urdf/asmHand.urdf.xacro" /> -->
+<xacro:include filename="$(find inmoov_description)/urdf/asmHead.urdf.xacro" />
+<xacro:include filename="$(find inmoov_description)/urdf/asmEye.urdf.xacro" />
+<xacro:include filename="$(find inmoov_description)/urdf/asmFace.urdf.xacro" />
+<xacro:include filename="$(find inmoov_description)/urdf/asmArm.urdf.xacro" />
+<xacro:include filename="$(find inmoov_description)/urdf/asmHand.urdf.xacro" />
+<!-- For now we start with a world link.  This is because we have no legs yet -->
+<!-- We are basically treating this as a stationary robot with a solid base -->
+<!-- rather than a mobile robot.  A mobile robot will start with a "base_link" instead -->
+<!-- The source I copied already has a base_link.  Maybe we start there later. -->
+<!-- For now we will leave it as part of the robot and leave world as well  -->
+<!-- We will change this later. -->
+<!--  -->
   <link name="world"/>
   <joint name="fixed" type="fixed">
@@ -19,12 +27,7 @@
   </joint>
   <link name="base_link">
-    <collision>
-      <geometry>
-        <cylinder length="0.11" radius="1.26"/>
-      </geometry>
-    </collision>
     <visual>
       <geometry>
-        <cylinder length="0.11" radius="1.26"/>
+        <cylinder length="0.11" radius="0.26"/>
       </geometry>
       <origin rpy="0 0 0" xyz="0 0 0.055"/>
@@ -46,11 +49,22 @@
     </visual>
   </link>
+  <link name="head_tilt_link">
+    <visual>
+      <geometry>
+        <mesh filename="package://inmoov_meshes/meshes/virtual.stl" scale="0.001 0.001 0.001"/>
+      </geometry>
+      <origin rpy="0 0 3.1415" xyz="0 0 0"/>
+      <xacro:frame_color/>
+    </visual>
+    <xacro:virtual_inertial/>
+  </link>
   <joint name="pedestal_to_mid_stomach_joint" type="fixed">
     <parent link="pedestal_link"/>
     <child link="mid_stomach_link"/>
-    <origin rpy="0 0 0"  xyz="0 0 0"/>
+     <origin rpy="0 0 0"  xyz="0 0 0"/>
   </joint>
+  <!-- Run macro called "torso" in file asmTorso.urdf.xacro -->
   <xacro:torso covers="yes" />
-  <!-- <joint name="head_roll_joint" type="revolute">
+  <joint name="head_roll_joint" type="revolute">
    <axis xyz="1 0 0"/>
    <limit effort="1000.0" lower="${head_roll_joint_lower}" upper="${head_roll_joint_upper}" velocity="${head_roll_joint_velocity}" />
@@ -66,5 +80,7 @@
    <child link="head_base_link"/>
   </joint>
+  <!-- Run macro called "head" in file asmHead.urdf.xacro -->
   <xacro:head covers="yes" />
+  <!-- Run macro called "face" in file asmFace.urdf.xacro -->
   <xacro:face covers="yes" />
   <joint name="face_joint" type="fixed">
@@ -73,4 +89,6 @@
     <child link="face_link"/>
   </joint>
+  <!-- Run macro called "face" in file asmArm.urdf.xacro -->
+  <!-- We pass the param "side" in order to process 2 arms with 2 hands, right(r) in this case-->
   <xacro:arm side="r" flip="1" covers="yes" />
   <joint name="r_shoulder_out_joint" type="revolute">
@@ -90,4 +108,6 @@
   </joint>
   <xacro:arm side="l" flip="-1" covers="yes" />
+  <!-- Run macro called "face" in file asmArm.urdf.xacro -->
+  <!-- We pass the param "side" in order to process 2 arms with 2 hands, left(l) in this case-->
   <joint name="l_shoulder_out_joint" type="revolute">
    <axis xyz="1 0 0"/>
@@ -104,4 +124,4 @@
    <parent link="l_forearm_link"/>
    <child link="l_hand_link"/>
-  </joint> -->
+  </joint>
 </robot>

File: src/inmoov_description/urdf/asmTorso.urdf.xacro (robot description, xacro)
@@ -3,14 +3,14 @@
 <xacro:macro name="torso" params="covers">
   <link name="mid_stomach_link">
+    <xacro:mid_stomach_inertial/>
     <visual>
       <geometry>
-        <mesh filename="package://inmoov_meshes/meshes/mid_stomach.stl" scale="0.001 0.001 0.001"/>
+        <cylinder length="0.94" radius="0.254"/>
       </geometry>
       <origin rpy="0 0 0" xyz="0 0 1.152"/>
       <xacro:frame_color/>
     </visual>
-    <xacro:mid_stomach_inertial/>
   </link>
-  <link name="disk_link">
+  <!-- <link name="disk_link">
     <visual>
       <geometry>
@@ -21,16 +21,16 @@
     </visual>
     <xacro:disk_inertial/>
-  </link>
+  </link> -->
   <link name="top_stomach_link">
     <visual>
       <geometry>
-        <mesh filename="package://inmoov_meshes/meshes/top_stomach.stl" scale="0.001 0.001 0.001"/>
+        <cylinder length="0.94" radius="0.254"/>
       </geometry>
-      <origin rpy="0 0 0" xyz="0 0 0"/>
+      <origin rpy="0 0 0" xyz="0 0 3"/>
       <xacro:frame_color/>
     </visual>
     <xacro:top_stomach_inertial/>
   </link>
-  <link name="torso_link">
+  <!-- <link name="torso_link">
     <visual>
       <geometry>
@@ -41,6 +41,6 @@
     </visual>
     <xacro:torso_inertial/>
-  </link>
-  <link name="kinect2_link">
+  </link> -->
+  <!-- <link name="kinect2_link">
     <visual>
       <geometry>
@@ -51,6 +51,6 @@
     </visual>
     <xacro:kinectone_inertial/>
-  </link>
-  <link name="kinect2_ir_optical_frame">
+  </link> -->
+  <!-- <link name="kinect2_ir_optical_frame">
     <visual>
       <geometry>
@@ -61,6 +61,6 @@
     </visual>
     <xacro:kinectone_inertial/>
-  </link>
-  <link name="kinect2_rgb_optical_frame">
+  </link> -->
+  <!-- <link name="kinect2_rgb_optical_frame">
     <visual>
       <geometry>
@@ -71,6 +71,6 @@
     </visual>
     <xacro:kinectone_inertial/>
-  </link>
-  <link name="chestplate_link">
+  </link> -->
+  <!-- <link name="chestplate_link">
     <visual>
       <geometry>
@@ -81,5 +81,5 @@
     </visual>
     <xacro:chest_inertial/>
-  </link>
+  </link> -->
   <joint name="waist_pan_joint" type="revolute">
    <axis xyz="0 0 1"/>
@@ -89,9 +89,10 @@
     <child link="top_stomach_link"/>
   </joint>
-  <joint name="disk_joint" type="fixed">
+  <!-- <joint name="disk_joint" type="fixed">
       <origin rpy="0 0 0" xyz="0.046 0 0.09"/>
     <parent link="top_stomach_link"/>
     <child link="disk_link"/>
-  </joint>
+  </joint> -->
+<!--
   <joint name="waist_roll_joint" type="revolute">
    <axis xyz="1 0 0"/>
@@ -120,5 +121,5 @@
     <parent link="torso_link"/>
     <child link="kinect2_rgb_optical_frame"/>
-  </joint>
+  </joint> -->
 </xacro:macro>
 </robot>
