Commit message: mvoed meshes

File: src/inmoov_description/robots/asmTorso.urdf.xacro (robot description, xacro)
@@ -1,5 +1,6 @@
 <?xml version="1.0"?>
-<robot name="inmoov" xmlns:xacro="http://ros.org/wiki/xacro">
-<xacro:macro name="torso" params="covers">
+<robot xmlns:xacro="http://ros.org/wiki/xacro">
+<xacro:macro name="torso">
+<!-- <xacro:macro name="torso" params="covers"> -->
   <link name="mid_stomach_link">
     <xacro:mid_stomach_inertial/>

File: src/inmoov_description/robots/inmoov.urdf.xacro (robot description, xacro)
@@ -7,5 +7,5 @@
 <!-- The following includes are for the various appendages -->
 <!-- <xacro:include filename="$(find inmoov_description)/urdf/asmBase.urdf.xacro" /> -->
-<xacro:include filename="$(find inmoov_description)/urdf/asmTorso.urdf.xacro" />
+<xacro:include filename="$(find inmoov_description)/robots/asmTorso.urdf.xacro" />
 <!-- <xacro:include filename="$(find inmoov_description)/urdf/asmHead.urdf.xacro" /> -->
 <!-- <xacro:include filename="$(find inmoov_description)/urdf/asmEye.urdf.xacro" /> -->
@@ -46,10 +46,10 @@
     </visual>
   </link>
+  <xacro:torso />
   <joint name="pedestal_to_mid_stomach_joint" type="fixed">
     <parent link="pedestal_link"/>
     <child link="mid_stomach_link"/>
-    <origin rpy="0 0 0"  xyz="0 0 0"/>
+    <origin rpy="0 0 0" xyz="0 0 0"/>
   </joint>
-  <xacro:torso covers="yes" />
   <!-- <joint name="head_roll_joint" type="revolute">
    <axis xyz="1 0 0"/>

File: src/inmoov_description/robots/inmoov_right_hand.urdf.xacro (robot description, xacro)
@@ -18,7 +18,7 @@
   <xacro:hand side="r" flip="1" covers="yes" />
   <joint name="base_to_hand_joint" type="revolute">
-   <axis xyz="0 0 1"/>
-<limit effort="1000.0" lower="-3.14" upper="0" velocity="0.5"/>
-<origin rpy="0 0 0" xyz="0 0 0"/>
+    <axis xyz="0 0 1"/>
+    <limit effort="1000.0" lower="-3.14" upper="0" velocity="0.5"/>
+    <origin rpy="0 0 0" xyz="0 0 0"/>
     <parent link="base_link"/>
     <child link="r_hand_link"/>
